File: pcb/rgb-digit/rgb-digit.kicad_pcb (KiCad board)
At the start: 2 copper layers, 22.9 x 39.4 mm, 26 parts, among them J1 5V IN, J2 GND IN, J3 5V OUT, J4 GND OUT, J5 DATA IN, J6 DATA OUT, U1 WS2812B, U2 WS2812B, U3 WS2812B, U4 WS2812B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

Commit message: Updated schematic of rgb-digits pcb * Changed sheet size to US letter * Added gerber and pdf files of each layers
Parts:
- added REF**: VAL**, Symbols:Gauge-XY-100mm, F.Cu at (102.9, 142.9)
Changed lines of the file:
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@@
-(kicad_pcb (version 4) (host pcbnew "(2016-03-01 BZR 6238)-product")
+(kicad_pcb (version 4) (host pcbnew "(2016-05-03 BZR 6266)-product")
   (general
-    (links 56)
+    (links 0)
     (no_connects 0)
-    (area 128.780915 84.32258 152.8598 124.764802)
+    (area 128.870915 84.41258 152.9598 124.764802)
     (thickness 1.6)
     (drawings 122)
     (tracks 204)
     (zones 0)
-    (modules 26)
+    (modules 27)
     (nets 11)
   )
-  (page A4)
+  (page USLetter)
   (title_block
     (title "Display - RGB Seven Seg. Digit")
@@
     (40 Dwgs.User user)
     (41 Cmts.User user)
-    (42 Eco1.User user hide)
+    (42 Eco1.User user)
     (43 Eco2.User user)
     (44 Edge.Cuts user)
@@
     )
   )
+  (module Symbols:Gauge-XY-100mm (layer F.Cu)
+    (at 102.87 142.875)
+    (descr "Gauge, Massstab, 100mm, SilkScreenTop, Type 1,")
+    (tags "Gauge, Massstab, 100mm, SilkScreenTop, Type 1,")
+    (fp_text reference REF** (at 0 3.81) (layer Eco1.User) hide
+      (effects (font (size 0.5 0.5) (thickness 0.1)))
+    )
+    (fp_text value VAL** (at 0 4.445) (layer Eco1.User) hide
+      (effects (font (size 0.5 0.5) (thickness 0.1)))
+    )
+    (fp_line (start 0 -9.99998) (end -1.99898 -9.99998) (layer Eco1.User) (width 0.15))
+    (fp_line (start 0 0) (end 0 -9.99998) (layer Eco1.User) (width 0.15))
+    (fp_line (start 0 0) (end -1.99898 0) (layer Eco1.User) (width 0.15))
+    (fp_line (start 0 -5.00126) (end -1.99898 -5.00126) (layer Eco1.User) (width 0.15))
+    (fp_line (start 0 -1.00076) (end -1.00076 -1.00076) (layer Eco1.User) (width 0.15))
+    (fp_line (start 0 -1.99898) (end -1.00076 -1.99898) (layer Eco1.User) (width 0.15))
+    (fp_line (start 0 -2.99974) (end -1.00076 -2.99974) (layer Eco1.User) (width 0.15))
+    (fp_line (start 0 -4.0005) (end -1.00076 -4.0005) (layer Eco1.User) (width 0.15))
+    (fp_line (start 0 -5.99948) (end -1.00076 -5.99948) (layer Eco1.User) (width 0.15))
+    (fp_line (start 0 -7.00024) (end -1.00076 -7.00024) (layer Eco1.User) (width 0.15))
+    (fp_line (start 0 -8.001) (end -1.00076 -8.001) (layer Eco1.User) (width 0.15))
+    (fp_line (start 0 -8.99922) (end -1.00076 -8.99922) (layer Eco1.User) (width 0.15))
+    (fp_text user 10mm (at -2.70002 -9.99998 270) (layer Eco1.User)
+      (effects (font (size 1 1) (thickness 0.15)))
+    )
+    (fp_text user 0 (at -2.79908 0 270) (layer Eco1.User)
+      (effects (font (size 1 1) (thickness 0.15)))
+    )
+    (fp_text user 5 (at -2.90068 -4.99872 270) (layer Eco1.User)
+      (effects (font (size 1 1) (thickness 0.15)))
+    )
+    (fp_line (start 0 -99.9998) (end -1.99898 -99.9998) (layer Eco1.User) (width 0.15))
+    (fp_line (start 0 -9.99998) (end 0 -99.9998) (layer Eco1.User) (width 0.15))
+    (fp_line (start 0 -15.00124) (end -1.00076 -15.00124) (layer Eco1.User) (width 0.15))
+    (fp_line (start 0 -19.99996) (end -1.99898 -19.99996) (layer Eco1.User) (width 0.15))
+    (fp_line (start 0 -25.00122) (end -1.00076 -25.00122) (layer Eco1.User) (width 0.15))
+    (fp_line (start 0 -29.99994) (end -1.99898 -29.99994) (layer Eco1.User) (width 0.15))
+    (fp_line (start 0 -35.0012) (end -1.00076 -35.0012) (layer Eco1.User) (width 0.15))
+    (fp_line (start 0 -39.99992) (end -1.99898 -39.99992) (layer Eco1.User) (width 0.15))
+    (fp_line (start 0 -45.00118) (end -1.00076 -45.00118) (layer Eco1.User) (width 0.15))
+    (fp_line (start 0 -49.9999) (end -1.99898 -49.9999) (layer Eco1.User) (width 0.15))
+    (fp_line (start 0 -55.00116) (end -1.00076 -55.00116) (layer Eco1.User) (width 0.15))
+    (fp_line (start 0 -59.99988) (end -1.99898 -59.99988) (layer Eco1.User) (width 0.15))
+    (fp_line (start 0 -65.00114) (end -1.00076 -65.00114) (layer Eco1.User) (width 0.15))
+    (fp_line (start 0 -69.99986) (end -1.99898 -69.99986) (layer Eco1.User) (width 0.15))
+    (fp_line (start 0 -75.00112) (end -1.00076 -75.00112) (layer Eco1.User) (width 0.15))
+    (fp_line (start 0 -79.99984) (end -1.99898 -79.99984) (layer Eco1.User) (width 0.15))
+    (fp_line (start 0 -85.0011) (end -1.00076 -85.0011) (layer Eco1.User) (width 0.15))
+    (fp_line (start 0 -89.99982) (end -1.99898 -89.99982) (layer Eco1.User) (width 0.15))
+    (fp_line (start 0 -95.00108) (end -1.00076 -95.00108) (layer Eco1.User) (width 0.15))
+    (fp_text user 20 (at -2.90068 -20.09902 270) (layer Eco1.User)
+      (effects (font (size 1 1) (thickness 0.15)))
+    )
+    (fp_text user 30 (at -2.99974 -29.99994 270) (layer Eco1.User)
+      (effects (font (size 1 1) (thickness 0.15)))
+    )
+    (fp_text user 40 (at -3.10134 -39.99992 270) (layer Eco1.User)
+      (effects (font (size 1 1) (thickness 0.15)))
+    )
+    (fp_text user 50 (at -3.10134 -49.9999 270) (layer Eco1.User)
+      (effects (font (size 1 1) (thickness 0.15)))
+    )
+    (fp_text user 60 (at -3.10134 -59.99988 270) (layer Eco1.User)
+      (effects (font (size 1 1) (thickness 0.15)))
+    )
+    (fp_text user 70 (at -3.302 -69.99986 270) (layer Eco1.User)
+      (effects (font (size 1 1) (thickness 0.15)))
+    )
+    (fp_text user 80 (at -3.40106 -79.99984 270) (layer Eco1.User)
+      (effects (font (size 1 1) (thickness 0.15)))
+    )
+    (fp_text user 90 (at -3.20294 -90.10142 270) (layer Eco1.User)
+      (effects (font (size 1 1) (thickness 0.15)))
+    )
+    (fp_text user 100mm (at -3.20294 -100.1014 270) (layer Eco1.User)
+      (effects (font (size 1 1) (thickness 0.15)))
+    )
+    (fp_text user 100mm (at 100.1014 3.20294) (layer Eco1.User)
+      (effects (font (size 1 1) (thickness 0.15)))
+    )
+    (fp_text user 90 (at 90.10142 3.20294) (layer Eco1.User)
+      (effects (font (size 1 1) (thickness 0.15)))
+    )
+    (fp_text user 80 (at 79.99984 3.40106) (layer Eco1.User)
+      (effects (font (size 1 1) (thickness 0.15)))
+    )
+    (fp_text user 70 (at 69.99986 3.302) (layer Eco1.User)
+      (effects (font (size 1 1) (thickness 0.15)))
+    )
+    (fp_text user 60 (at 59.99988 3.10134) (layer Eco1.User)
+      (effects (font (size 1 1) (thickness 0.15)))
+    )
+    (fp_text user 50 (at 49.9999 3.10134) (layer Eco1.User)
+      (effects (font (size 1 1) (thickness 0.15)))
+    )
+    (fp_text user 40 (at 39.99992 3.10134) (layer Eco1.User)
+      (effects (font (size 1 1) (thickness 0.15)))
+    )
+    (fp_text user 30 (at 29.99994 2.99974) (layer Eco1.User)
+      (effects (font (size 1 1) (thickness 0.15)))
+    )
+    (fp_text user 20 (at 20.09902 2.90068) (layer Eco1.User)
+      (effects (font (size 1 1) (thickness 0.15)))
+    )
+    (fp_line (start 95.00108 0) (end 95.00108 1.00076) (layer Eco1.User) (width 0.15))
+    (fp_line (start 89.99982 0) (end 89.99982 1.99898) (layer Eco1.User) (width 0.15))
+    (fp_line (start 85.0011 0) (end 85.0011 1.00076) (layer Eco1.User) (width 0.15))
+    (fp_line (start 79.99984 0) (end 79.99984 1.99898) (layer Eco1.User) (width 0.15))
+    (fp_line (start 75.00112 0) (end 75.00112 1.00076) (layer Eco1.User) (width 0.15))
+    (fp_line (start 69.99986 0) (end 69.99986 1.99898) (layer Eco1.User) (width 0.15))
+    (fp_line (start 65.00114 0) (end 65.00114 1.00076) (layer Eco1.User) (width 0.15))
+    (fp_line (start 59.99988 0) (end 59.99988 1.99898) (layer Eco1.User) (width 0.15))
+    (fp_line (start 55.00116 0) (end 55.00116 1.00076) (layer Eco1.User) (width 0.15))
+    (fp_line (start 49.9999 0) (end 49.9999 1.99898) (layer Eco1.User) (width 0.15))
+    (fp_line (start 45.00118 0) (end 45.00118 1.00076) (layer Eco1.User) (width 0.15))
+    (fp_line (start 39.99992 0) (end 39.99992 1.99898) (layer Eco1.User) (width 0.15))
+    (fp_line (start 35.0012 0) (end 35.0012 1.00076) (layer Eco1.User) (width 0.15))
+    (fp_line (start 29.99994 0) (end 29.99994 1.99898) (layer Eco1.User) (width 0.15))
+    (fp_line (start 25.00122 0) (end 25.00122 1.00076) (layer Eco1.User) (width 0.15))
+    (fp_line (start 19.99996 0) (end 19.99996 1.99898) (layer Eco1.User) (width 0.15))
+    (fp_line (start 15.00124 0) (end 15.00124 1.00076) (layer Eco1.User) (width 0.15))
+    (fp_line (start 9.99998 0) (end 99.9998 0) (layer Eco1.User) (width 0.15))
+    (fp_line (start 99.9998 0) (end 99.9998 1.99898) (layer Eco1.User) (width 0.15))
+    (fp_text user 5 (at 4.99872 2.90068) (layer Eco1.User)
+      (effects (font (size 1 1) (thickness 0.15)))
+    )
+    (fp_text user 0 (at 0 2.79908) (layer Eco1.User)
+      (effects (font (size 1 1) (thickness 0.15)))
+    )
+    (fp_text user 10mm (at 9.99998 2.70002) (layer Eco1.User)
+      (effects (font (size 1 1) (thickness 0.15)))
+    )
+    (fp_line (start 8.99922 0) (end 8.99922 1.00076) (layer Eco1.User) (width 0.15))
+    (fp_line (start 8.001 0) (end 8.001 1.00076) (layer Eco1.User) (width 0.15))
+    (fp_line (start 7.00024 0) (end 7.00024 1.00076) (layer Eco1.User) (width 0.15))
+    (fp_line (start 5.99948 0) (end 5.99948 1.00076) (layer Eco1.User) (width 0.15))
+    (fp_line (start 4.0005 0) (end 4.0005 1.00076) (layer Eco1.User) (width 0.15))
+    (fp_line (start 2.99974 0) (end 2.99974 1.00076) (layer Eco1.User) (width 0.15))
+    (fp_line (start 1.99898 0) (end 1.99898 1.00076) (layer Eco1.User) (width 0.15))
+    (fp_line (start 1.00076 0) (end 1.00076 1.00076) (layer Eco1.User) (width 0.15))
+    (fp_line (start 5.00126 0) (end 5.00126 1.99898) (layer Eco1.User) (width 0.15))
+    (fp_line (start 0 0) (end 0 1.99898) (layer Eco1.User) (width 0.15))
+    (fp_line (start 0 0) (end 9.99998 0) (layer Eco1.User) (width 0.15))
+    (fp_line (start 9.99998 0) (end 9.99998 1.99898) (layer Eco1.User) (width 0.15))
+  )
   (gr_line (start 134.874 117.475) (end 135.382 116.967) (layer Eco1.User) (width 0.2))
