File: fab-files/pcb-panels/display/panel-display.kicad_pcb (KiCad board)
At the start: 2 copper layers, 99.1 x 95.2 mm, 218 parts, among them J1 5V IN, J1 DATA IN, J1 HEADER-1x05, J1 HEADER-1x06, J2 5V IN, J2 GND IN, J2 HEADER-1x01, J3 5V OUT, J3 GND IN, J3 HEADER-1x01, J4 5V OUT, J4 GND OUT, J4 HEADER-1x01, J5 DATA IN, J5 GND OUT, J5 HEADER-1x01, J6 DATA OUT, Q1 BSS138, Q2 BSS138, SW1 ALARM, SW2 MENU, SW3 SET, U1 AT42QT1070, U1 ER-OLED1602-4W, U1 TSL2561, U1 WS2812B, U2 LP2981, U2 LT1109CS8-12, U2 WS2812B, U3 WS2812B, U4 WS2812B, U5 WS2812B, U6 WS2812B, U7 WS2812B

Commit message: Updated display pcb panel
Parts:
- added R8: 10k, SMT:R-0603, F.Cu at (127.6, 78.1)
- R1: value 500k -> 470k
- moved U1 0.64 mm to (185.4, 69.6)
Connections:
- net /RESET renamed /~RESET
Routing:
- net +5V: track 355.3 -> 362.3 mm
- net /~RESET: track 51.2 -> 58.1 mm, vias 2 -> 3
- net GND: track 392.9 -> 394.0 mm, vias 161 -> 162
- net Net-(R1-Pad1): track 27.8 -> 27.2 mm
- net +3V3: track 58.9 -> 58.2 mm
- net /SCL_3V3: track 26.4 -> 27.0 mm
- net /INT: track 15.4 -> 16.1 mm
- net /SDA_3V3: track 33.9 -> 34.5 mm
Other:
- net class Default: clearance 0.3048 -> 0.254
- net class Power: clearance 0.4064 -> 0.254; trace_width 0.4064 -> 0.3048; via_dia 1.27 -> 1.1684
- rule trace_clearance: 0.3048 -> 0.254
