File: pcb/alarm-switch/alarm-switch.kicad_pcb (KiCad board)
At the start: 2 copper layers, 33 x 16.5 mm, 4 parts, among them J1 HEADER-1x03, SW1 L102011ML04Q

Commit message: Updated PCB design
+ Completed daughterboard PCB layout.
* Corrected soldermask clerance on front panel pcb.
- Removed input resistor on DIN for RGB lamp board.
* Modified PCB layout for PSU board.
* Updated gerber files.
* Updated schematics pdf, BOM.
Parts:
- SW1: footprint switches:CK_L102XXXML04 -> switches:CK-L102XXXML04
Changed lines of the file:
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@@
-(kicad_pcb (version 4) (host pcbnew 4.0.7-e2-6376~60~ubuntu17.10.1)
+(kicad_pcb (version 20171130) (host pcbnew 5.0.0-fee4fd1~65~ubuntu17.10.1)
   (general
-    (links 16)
-    (no_connects 4)
-    (area 107.239999 91.999999 140.410001 108.660001)
     (thickness 1.6)
     (drawings 9)
@@
       (layerselection 0x00030_80000001)
       (usegerberextensions false)
+      (usegerberattributes false)
+      (usegerberadvancedattributes false)
+      (creategerberjobfile false)
       (excludeedgelayer true)
       (linewidth 0.100000)
@@
       (hpglpennumber 1)
       (hpglpenspeed 20)
-      (hpglpendiameter 15)
-      (hpglpenoverlay 2)
+      (hpglpendiameter 15.000000)
       (psnegative false)
       (psa4output false)
@@
     (add_net "Net-(J1-Pad2)")
     (add_net "Net-(J1-Pad3)")
+  )
+  (module switches:CK-L102XXXML04 (layer F.Cu)
+    (at 123.825 108.585)
+    (descr "C&K Slide switch - SPDT - R/A TH")
+    (tags "slide switch")
+    (fp_text reference SW1 (at -9.779 -10.541) (layer F.SilkS)
+      (effects (font (size 1 1) (thickness 0.18)) (justify left bottom))
+    )
+    (fp_text value L102011ML04Q (at 0 1.72) (layer F.SilkS) hide
+      (effects (font (size 1 1) (thickness 0.15)))
+    )
+    (fp_line (start -10.668 1.016) (end 10.668 1.016) (layer F.CrtYd) (width 0.05))
+    (fp_line (start 10.668 -11.176) (end 10.668 1.016) (layer F.CrtYd) (width 0.05))
+    (fp_line (start -10.668 -11.176) (end 10.668 -11.176) (layer F.CrtYd) (width 0.05))
+    (fp_line (start -10.668 -11.176) (end -10.668 1.016) (layer F.CrtYd) (width 0.05))
+    (fp_line (start -9.652 0) (end 9.652 0) (layer F.SilkS) (width 0.18))
+    (fp_line (start 9.652 0) (end 9.652 -10.16) (layer F.SilkS) (width 0.18))
+    (fp_line (start 9.652 -10.16) (end -9.652 -10.16) (layer F.SilkS) (width 0.18))
+    (fp_line (start -9.652 -10.16) (end -9.652 0) (layer F.SilkS) (width 0.18))
+    (fp_line (start -0.635 -10.16) (end -0.635 -11.303) (layer F.SilkS) (width 0.18))
+    (fp_line (start 0.635 -10.16) (end 0.635 -11.303) (layer F.SilkS) (width 0.18))
+    (fp_arc (start 0 -11.303) (end -0.635 -11.303) (angle 180) (layer F.SilkS) (width 0.18))
+    (pad 3 thru_hole circle (at 4.7498 -7.62) (size 3.048 3.048) (drill 1.651) (layers *.Cu *.Mask)
+      (net 4 "Net-(J1-Pad3)"))
+    (pad 2 thru_hole circle (at 0 -7.62) (size 3.048 3.048) (drill 1.651) (layers *.Cu *.Mask)
+      (net 3 "Net-(J1-Pad2)"))
+    (pad 1 thru_hole circle (at -4.7498 -7.62) (size 3.048 3.048) (drill 1.651) (layers *.Cu *.Mask)
+      (net 2 "Net-(J1-Pad1)"))
+    (model ${KISYS3DMOD}/switches.pretty/CK-L102XXXML04.wrl
+      (at (xyz 0 0 0))
+      (scale (xyz 1 1 1))
+      (rotate (xyz 0 0 0))
+    )
   )
   (module conn-wire-pads:Hole-Screw-#4 (layer F.Cu)
@@
     )
   )
-  (module switches:CK_L102XXXML04 (layer F.Cu)
-    (at 123.825 108.585)
-    (descr "C&K Slide switch - SPDT - R/A TH")
-    (tags "slide switch")
-    (fp_text reference SW1 (at -9.779 -10.541) (layer F.SilkS)
-      (effects (font (size 1 1) (thickness 0.18)) (justify left bottom))
-    )
-    (fp_text value L102011ML04Q (at -7.62 1.016) (layer F.SilkS) hide
-      (effects (font (size 1 1) (thickness 0.15)))
-    )
-    (fp_arc (start 0 -11.303) (end -0.635 -11.303) (angle 180) (layer F.SilkS) (width 0.18))
-    (fp_line (start 0.635 -10.16) (end 0.635 -11.303) (layer F.SilkS) (width 0.18))
-    (fp_line (start -0.635 -10.16) (end -0.635 -11.303) (layer F.SilkS) (width 0.18))
-    (fp_line (start -9.652 -10.16) (end -9.652 0) (layer F.SilkS) (width 0.18))
-    (fp_line (start 9.652 -10.16) (end -9.652 -10.16) (layer F.SilkS) (width 0.18))
-    (fp_line (start 9.652 0) (end 9.652 -10.16) (layer F.SilkS) (width 0.18))
-    (fp_line (start -9.652 0) (end 9.652 0) (layer F.SilkS) (width 0.18))
-    (fp_line (start -10.668 -11.176) (end -10.668 1.016) (layer F.CrtYd) (width 0.05))
-    (fp_line (start -10.668 -11.176) (end 10.668 -11.176) (layer F.CrtYd) (width 0.05))
-    (fp_line (start 10.668 -11.176) (end 10.668 1.016) (layer F.CrtYd) (width 0.05))
-    (fp_line (start -10.668 1.016) (end 10.668 1.016) (layer F.CrtYd) (width 0.05))
-    (pad 1 thru_hole circle (at -4.7498 -7.62) (size 3.048 3.048) (drill 1.651) (layers *.Cu *.Mask)
-      (net 2 "Net-(J1-Pad1)"))
-    (pad 2 thru_hole circle (at 0 -7.62) (size 3.048 3.048) (drill 1.651) (layers *.Cu *.Mask)
-      (net 3 "Net-(J1-Pad2)"))
-    (pad 3 thru_hole circle (at 4.7498 -7.62) (size 3.048 3.048) (drill 1.651) (layers *.Cu *.Mask)
-      (net 4 "Net-(J1-Pad3)"))
-  )
   (gr_text PC-09 (at 123.825 105.41) (layer B.SilkS)
