File: pcb/daughterboard/daughterboard.sch (KiCad schematic (older format))
At the start: 0 parts

Commit message: Revised touch and front panel PCB, Added Motherboard PCB
Parts:
- added H1: HEADER-1x01, conn-wire-pads:SolderPad-100x500, symbol connectors:HEADER-1x01
- added H2: HEADER-1x01, conn-wire-pads:SolderPad-100x200, symbol connectors:HEADER-1x01
- added J1: LAMP, conn-header:DF3A-3P-2DSA, symbol connectors:HEADER-1x03
- added J2: DISPLAY, conn-header:DF3A-8P-2DSA, symbol connectors:HEADER-1x08
- added J3: SPKR, conn-header:DF3A-4P-2DSA, symbol connectors:HEADER-1x04
- added J4: MB I/O, conn-header:HDR-M-2x08, symbol connectors:HEADER-2x08
- added J5: PWR, conn-header:HDR-M-1x04, symbol connectors:HEADER-1x04
- added R1: 300, smt:R-0603, symbol passive:RESISTOR
Connections:
- net labels added: +3V3, +5V, A_SHDN, CD_CS, CD_RST, CD_XDCS, DREQ, GND, KPD_CHG, K_CHG, LED0, LED1, LED_SHDN, MISO, MOSI, RESET, SCLK, SCL_5V, SDA_5V, SUP_+5V, SUP_GND
- wire segments 0 -> 43
- no-connect marks 0 -> 2

Commit message: Updated PCB design
+ Completed daughterboard PCB layout.
* Corrected soldermask clerance on front panel pcb.
- Removed input resistor on DIN for RGB lamp board.
* Modified PCB layout for PSU board.
* Updated gerber files.
* Updated schematics pdf, BOM.
Parts:
- added C1, C10, C2, C26, C27, C29, C3, C30, C4, C5, C6, C7, C8, C9: 100nF, smt:C-0603, symbol passive:CAP
- added C11, C14, C16: 10uF 6V3, smt:CPL-0805, symbol passive:CAP-E
- added C12, C13: 20pF, smt:C-0603, symbol passive:CAP
- added C15, C20, C21, C22, C23: 1uF, smt:C-0805, symbol passive:CAP
- added C17: 47nF, smt:C-0603, symbol passive:CAP
- added C18, C19: 10nF, smt:C-0603, symbol passive:CAP
- added C24, C25, C28: 10uF, smt:C-0805, symbol passive:CAP
- added C31, C32, C33, C34: 1nF, smt:C-0603, symbol passive:CAP
- added J6: DB-C, conn-header:HDR-M-1x02, symbol connectors:HEADER-1x02
- added J7: ALARM SW, conn-header:DF3A-2P-2DSA, symbol connectors:HEADER-1x02
- added L1, L2: 2508053007Y0, smt:FER-0805, symbol passive:FERRITE
- added L3, L4, L5, L6: MPZ1608S221A, smt:FER-0603, symbol passive:FERRITE
- added Q1: NTF6P02, smt-sot:SOT-223, symbol transistor:NTF6P02
- added R10, R9: 20, smt:R-0603, symbol passive:RESISTOR
- added R11, R2, R7: 10k, smt:R-0603, symbol passive:RESISTOR
- added R12, R13, R14, R15, R16, R17, R18, R19, R4, R6: 100k, smt:R-0603, symbol passive:RESISTOR
- added R3: 470, smt:R-0603, symbol passive:RESISTOR
- added R5: 1M, smt:R-0603, symbol passive:RESISTOR
- added R8: 10, smt:R-0603, symbol passive:RESISTOR
- added TP1, TP10, TP2, TP3, TP4, TP5, TP6, TP7, TP8, TP9: TEST-POINT, conn-wire-pads:TEST-POINT-50, symbol connectors:TEST-POINT
- added U1: VS1053B, smt-qfp:QFP-7-48, symbol ic-misc:VS1053B
- added U2: 74AHC1G04SE-7, smt-sot:SOT-353, symbol ic-logic:74?1G04
- added U3: AP7312-1833W6, smt-sot:SOT23-6, symbol ic-power:AP7312-????W6
- added U4: TPA2016D2, smt-qfn:QFN20-EP-4x4, symbol ic-misc:TPA2016D2
- added U5: SN74LVC2G34DBV, smt-sot:SOT23-6, symbol ic-logic:74?2G34
- added Y1: 12.288 MHz, crystals:smt-CSM-3X-7x4mm, symbol passive:CRYSTAL
- H1: value HEADER-1x01 -> Solder pad 2; Family Connector -> Virtual
- H2: value HEADER-1x01 -> Solder Pad 2; Family Connector -> Virtual
- J1: Part - -> DF3A-3P-2DSA
- J2: Part - -> DF3A-8P-2DSA
- J3: Part - -> DF3A-4P-2DSA
- J4: value MB I/O -> DB-A; Family Connector -> Virtual
- J5: value PWR -> DB-B; Family Connector -> Virtual
- R1: value 300 -> 470
Connections:
- net labels added: +1V8, AGND, ALRM_SW, AVDD, CCS_3V3, CMOSI_3V3, CRST_3V3, GBUF, GPIO0, GPIO1, GPIO2, GPIO3, GPIO4, GPIO5, GPIO6, GPIO7, KCHG, LEFT, OUT_L+, OUT_L-, OUT_R+, OUT_R-, PIX_CLK, PIX_LAMP, PIX_SHDN, PIX_VCC, RIGHT, SCL, SCLK_3V3, SDA, SUP_AGND, SUP_AVDD, XDCS_3V3
- net labels removed: CD_CS, CD_RST, CD_XDCS, KPD_CHG, K_CHG, LED0, LED1, LED_SHDN, MOSI, RESET, SCLK, SCL_5V, SDA_5V
- wire segments 43 -> 347
- no-connect marks 2 -> 7
Other:
- note added: "I2C Addr. : 0xB0"
