File: pcb/prototype/display-adapter/display-adapter.sch (KiCad schematic (older format))
At the start: 5 parts, among them J1 HEADER-1x08, J2 HEADER-1x02, J3 HEADER-1x02, J4 HEADER-1x03, J5 HEADER-1x05

Commit message: Updated PCB design
+ Completed daughterboard PCB layout.
* Corrected soldermask clerance on front panel pcb.
- Removed input resistor on DIN for RGB lamp board.
* Modified PCB layout for PSU board.
* Updated gerber files.
* Updated schematics pdf, BOM.
Parts:
- removed J1: HEADER-1x08, conn-header:DF3A-8P-2DSA, symbol HEADER-1x08
- removed J4: HEADER-1x03, conn-header:DF3A-3P-2DSA, symbol HEADER-1x03
- removed J5: HEADER-1x05, conn-header:HDR-M-1x05, symbol HEADER-1x05
- added C1: 100nF, smt:C-0603, symbol passive:CAP
- added J1: DISPLAY, conn-header:DF3A-8P-2DSA, symbol connectors:HEADER-1x08
- added J4: LAMP, conn-header:DF3A-3P-2DSA, symbol connectors:HEADER-1x03
- added J5: HEADER-1x06, conn-header:HDR-M-1x06, symbol connectors:HEADER-1x06
- added Q1: NTF6P02, smt-sot:SOT-223, symbol transistor:NTF6P02
- added R1: 10k, smt:R-0603, symbol passive:RESISTOR
- added R2, R3: 470, smt:R-0603, symbol passive:RESISTOR
- added U1: SN74LVC2G34DBV, smt-sot:SOT23-6, symbol ic-logic:74?2G34
- J2, J3: symbol HEADER-1x02 -> display-adapter-rescue:HEADER-1x02
Connections:
- net labels added: KCHG, PIX_CLK, PIX_LAMP, PIX_SHDN, PIX_VCC, SCL, SDA
- wire segments 31 -> 48
Other:
- moved on the sheet: J2, J3
