File: pcb/rgb-lamp/rgb-lamp.sch (KiCad schematic (older format))
At the start: 10 parts, among them J1 HEADER-1x03, U1 WS2812B, U2 WS2812B, U3 WS2812B

Commit message: Replaced RGB leds with IN-PI554FCH instead of WS2812B
Parts:
- U1, U2, U3: value WS2812B -> IN-PI554FCH
Changed lines of the file:
@@
 Sheet 1 1
 Title "RGB Lamp"
-Date "2018-08-13"
+Date "2018-08-29"
 Rev "A"
 Comp ""
@@
 P 5200 3750
 F 0 "U1" H 4850 4050 60  0000 L BNB
-F 1 "WS2812B" H 4850 3450 40  0000 L TNN
+F 1 "IN-PI554FCH" H 4850 3450 40  0000 L TNN
 F 2 "smt:LED-5050" H 4850 3375 40  0001 L TNN
 F 3 "" H 4850 4050 50  0000 C CNN
@@
 P 6600 3750
 F 0 "U2" H 6250 4050 60  0000 L BNB
-F 1 "WS2812B" H 6250 3450 40  0000 L TNN
+F 1 "IN-PI554FCH" H 6250 3450 40  0000 L TNN
 F 2 "smt:LED-5050" H 6250 3375 40  0001 L TNN
 F 3 "" H 6250 4050 50  0000 C CNN
@@
 P 8000 3750
 F 0 "U3" H 7650 4050 60  0000 L BNB
-F 1 "WS2812B" H 7650 3450 40  0000 L TNN
+F 1 "IN-PI554FCH" H 7650 3450 40  0000 L TNN
 F 2 "smt:LED-5050" H 7650 3375 40  0001 L TNN
 F 3 "" H 7650 4050 50  0000 C CNN

Commit message: Updated PCB design
+ Completed daughterboard PCB layout.
* Corrected soldermask clerance on front panel pcb.
- Removed input resistor on DIN for RGB lamp board.
* Modified PCB layout for PSU board.
* Updated gerber files.
* Updated schematics pdf, BOM.
Parts:
- removed R1: 300, smt:R-0603, symbol passive:RESISTOR
Connections:
- wire segments 38 -> 37
