File: pcb/psu/psu.sch (KiCad schematic (older format))
At the start: 4 parts, among them J1 VIN, J2 HEADER-1x01, J3 HEADER-1x01, J4 SIGNAL

Commit message: Updated PCB design
+ Completed daughterboard PCB layout.
* Corrected soldermask clerance on front panel pcb.
- Removed input resistor on DIN for RGB lamp board.
* Modified PCB layout for PSU board.
* Updated gerber files.
* Updated schematics pdf, BOM.
Parts:
- removed J2: HEADER-1x01, conn-header:HDR-M-1x01, symbol connectors:HEADER-1x01
- removed J4: SIGNAL, conn-header:HDR-M-1x02, symbol connectors:HEADER-1x02
- added J2: HEADER-1x04, conn-header:HDR-M-1x04, symbol connectors:HEADER-1x04
- J1: Part - -> TSW-103-07-F-D
- J3: footprint conn-header:HDR-M-1x01 -> conn-wire-pads:Hole-Screw-#4; Family Virtual -> Connector
Connections:
- wire segments 12 -> 8
Changed lines of the file:
@@
 F 2 "conn-header:HDR-M-2x03" H 2700 2600 60  0001 C CNN
 F 3 "" H 2700 2600 60  0001 C CNN
-F 4 "-" H 2600 4100 40  0001 L BNN "Part"
+F 4 "TSW-103-07-F-D" H 2600 4100 40  0001 L BNN "Part"
 F 5 "Virtual" H 2600 4200 40  0001 L BNN "Family"
 	1    2700 3800
 	1    0    0    -1
 $EndComp
-$Comp
-L connectors:HEADER-1x02 J4
-U 1 1 5CA32EF2
-P 2850 5750
-F 0 "J4" H 2800 5900 60  0000 L BNB
-F 1 "SIGNAL" V 3000 5750 40  0000 C CNN
-F 2 "conn-header:HDR-M-1x02" H 2850 5750 60  0001 C CNN
-F 3 "" H 2850 5750 60  0001 C CNN
-F 4 "-" H 2800 6000 40  0001 L BNN "Part"
-F 5 "Virtual" H 2800 6100 40  0001 L BNN "Family"
-	1    2850 5750
-	1    0    0    -1
-$EndComp
-$Comp
-L connectors:HEADER-1x01 J2
-U 1 1 5CA32FAE
-P 2850 6450
-F 0 "J2" H 2800 6550 60  0000 L BNB
-F 1 "HEADER-1x01" V 3000 6450 40  0001 C CNN
-F 2 "conn-header:HDR-M-1x01" H 2700 6425 60  0001 C CNN
-F 3 "" H 2800 6525 60  0001 C CNN
-F 4 "-" H 2800 6650 40  0001 L BNN "Part"
-F 5 "Virtual" H 2800 6750 40  0001 L BNN "Family"
-	1    2850 6450
-	1    0    0    -1
-$EndComp
-$Comp
-L connectors:HEADER-1x01 J3
-U 1 1 5CA3303F
-P 2850 6800
-F 0 "J3" H 2800 6900 60  0000 L BNB
-F 1 "HEADER-1x01" V 3000 6800 40  0001 C CNN
-F 2 "conn-header:HDR-M-1x01" H 2700 6775 60  0001 C CNN
-F 3 "" H 2800 6875 60  0001 C CNN
-F 4 "-" H 2800 7000 40  0001 L BNN "Part"
-F 5 "Virtual" H 2800 7100 40  0001 L BNN "Family"
-	1    2850 6800
-	1    0    0    -1
-$EndComp
-$Comp
-L power:GND #PWR0101
-U 1 1 5CA3342F
-P 2600 7000
-F 0 "#PWR0101" H 2600 7050 30  0001 C CNN
-F 1 "GND" H 2600 6875 30  0001 C CNN
-F 2 "" H 2600 7000 60  0000 C CNN
-F 3 "" H 2600 7000 60  0000 C CNN
-	1    2600 7000
-	1    0    0    -1
-$EndComp
-Wire Wire Line
-	2700 6800 2600 6800
-Wire Wire Line
-	2600 6800 2600 7000
-Wire Wire Line
-	2700 6450 2600 6450
-Wire Wire Line
-	2600 6450 2600 6800
-Connection ~ 2600 6800
 $Comp
 L power:GND #PWR0102
@@
 Wire Wire Line
 	3250 3800 3250 3550
+$Comp
+L connectors:HEADER-1x04 J2
+U 1 1 5BA2EBB6
+P 3400 5100
+F 0 "J2" H 3350 5350 60  0000 L BNB
+F 1 "HEADER-1x04" V 3550 5100 40  0000 C CNN
+F 2 "conn-header:HDR-M-1x04" H 3400 5100 60  0001 C CNN
+F 3 "" H 3400 5100 60  0001 C CNN
+F 4 "TSW-104-07-F-S" H 3350 5450 40  0001 L BNN "Part"
+F 5 "Connector" H 3350 5550 40  0001 L BNN "Family"
+	1    3400 5100
+	-1   0    0    -1
+$EndComp
+$Comp
+L connectors:HEADER-1x01 J3
+U 1 1 5BA3D5A7
+P 1650 6600
+F 0 "J3" H 1600 6700 60  0000 L BNB
+F 1 "HEADER-1x01" V 1800 6600 40  0000 C CNN
+F 2 "conn-wire-pads:Hole-Screw-#4" H 1500 6575 60  0001 C CNN
+F 3 "" H 1600 6675 60  0001 C CNN
+F 4 "-" H 1600 6800 40  0001 L BNN "Part"
+F 5 "Connector" H 1600 6900 40  0001 L BNN "Family"
+	1    1650 6600
+	1    0    0    -1
+$EndComp
 $EndSCHEMATC

Commit message: PSU board schematics/layout
Parts:
- removed J3: HEADER-1x01, conn-wire-pads:Hole-Screw-#4, symbol connectors:HEADER-1x01
- added C1, C11, C12, C13, C2: 10uF, smt:C-0805, symbol passive:CAP
- added C10: 1uF, smt:C-0603, symbol passive:CAP
- added C3, C5: 10uF, smt:C-0603, symbol passive:CAP
- added C4: 100nF, smt:C-0603, symbol passive:CAP
- added C6, C7, C8: 22uF, smt:C-0805, symbol passive:CAP
- added C9: 470nF, smt:C-0603, symbol passive:CAP
- added D1: RED, smt:LED-0805, symbol opto:LED
- added H1: Hole, conn-wire-pads:Hole-Screw-#4, symbol connectors:Hole
- added J3: BATTERY, conn-jst:S2B-PH-K, symbol connectors:HEADER-1x02
- added L1: 1.5uH, smt-inductor:SPM5030-HZ, symbol passive:INDUCTOR
- added Q1, Q2: MMST3904, smt-sot:SOT23, symbol transistor:MMST3904
- added R1, R11, R13, R14, R15, R16: 10k, smt:R-0603, symbol passive:RESISTOR
- added R10: 0, smt:R-0603, symbol passive:RESISTOR
- added R12, R3, R4, R5, R6: 100k, smt:R-0603, symbol passive:RESISTOR
- added R17: 680, smt:R-0603, symbol passive:RESISTOR
- added R2: 0.01 1%, smt:R-1206, symbol passive:RESISTOR
- added R7: 787k, smt:R-0603, symbol passive:RESISTOR
- added R8: 5.6k, smt:R-0603, symbol passive:RESISTOR
- added R9: 1.1k, smt:R-0603, symbol passive:RESISTOR
- added TP1: VBAT, conn-wire-pads:TEST-POINT-50, symbol connectors:TEST-POINT
- added TP2: VIN, conn-wire-pads:TEST-POINT-50, symbol connectors:TEST-POINT
- added TP3: VSYS, conn-wire-pads:TEST-POINT-50, symbol connectors:TEST-POINT
- added TP4: GND, conn-wire-pads:TEST-POINT-50, symbol connectors:TEST-POINT
- added TP5: VOUT, conn-wire-pads:TEST-POINT-50, symbol connectors:TEST-POINT
- added U1: BQ27441-G1, smt-son:PDSO-N12, symbol ic-power:BQ27441-G1
- added U2: BQ24075, smt-qfn:QFN16-EP-3x3, symbol ic-power:BQ24075
- added U3: TPS630701, smt-qfn:VQFN15N, symbol ic-power:TPS63070
- J1: Family Virtual -> Connector
- J2: value HEADER-1x04 -> SIGNAL
Connections:
- net labels added: +BATT, +SYS, BATT_IN, L1, L2, ON_BATT, SCL, SDA, SUP_+BATT, SUP_+VIN, SUP_GND, SYSOFF, ~CHG
- wire segments 8 -> 182
- no-connect marks 0 -> 1
Other:
- note added: "C3 and C5 should be a 0603 capacitor and \nmust be located as close as possible to the IC."
- note added: "NOTE 1 :\n"
- moved on the sheet: J1, J2
